Commit message: bugfix : gripper is now fixed joint

File: src/macgyvbot_resources/urdf/m0609_onrobot_rg2_combined.urdf (robot description, URDF)
Before this commit: robot m0609, 17 links, 16 joints
Joints:
- joint finger_joint: axis -0.0 0.999949 -0.010122 -> (none); limit lower=0 upper=1.18 effort=50.0 velocity=2.0 -> (none); type revolute -> fixed
- joint left_inner_finger_joint: axis 0.0 -0.999949 0.010122 -> (none); limit lower=-1.19 upper=0.01 effort=50.0 velocity=2.0 -> (none); mimic joint=finger_joint multiplier=-1 offset=0 -> (none); type revolute -> fixed
- joint left_inner_knuckle_joint: axis -0.0 0.999949 -0.010122 -> (none); limit lower=-1.19 upper=0.01 effort=50.0 velocity=2.0 -> (none); mimic joint=finger_joint multiplier=-1 offset=0 -> (none); type revolute -> fixed
- joint left_outer_knuckle_joint: axis -0.0 0.999949 -0.010122 -> (none); limit lower=-1.19 upper=0.01 effort=50.0 velocity=2.0 -> (none); mimic joint=finger_joint multiplier=-1 offset=0 -> (none); type revolute -> fixed
- joint right_inner_finger_joint: axis 0.0 0.999949 -0.010122 -> (none); limit lower=-1.19 upper=0.01 effort=50.0 velocity=2.0 -> (none); mimic joint=finger_joint multiplier=-1 offset=0 -> (none); type revolute -> fixed
- joint right_inner_knuckle_joint: axis -0.0 0.999949 -0.010122 -> (none); limit lower=-0.01 upper=1.19 effort=50.0 velocity=2.0 -> (none); mimic joint=finger_joint multiplier=1 offset=0 -> (none); type revolute -> fixed
